Commit message: change urdf

File: arm_description/urdf/arm_description.urdf (robot description, URDF)
Before this commit: robot arm_description, 5 links, 4 joints
Joints:
- joint joint1: limit lower=0 upper=0.25 effort=50 velocity=1 -> lower=-0.24 upper=0 effort=50 velocity=1
- joint joint2: limit lower=-3.14 upper=3.14 effort=50 velocity=1 -> lower=-1.7 upper=1.7 effort=50 velocity=1
- joint joint3: limit lower=-3.14 upper=3.14 effort=50 velocity=1 -> lower=-3 upper=3 effort=50 velocity=1

Commit message: change moveit
对moveit生成的文件进行修改使得可以用rviz与gazebo联合仿真。
问题：demo.launch可以执行规划，但demo_gazebo.launch 却每一次规划都是从起点开始，暂时不清楚是为什么

File: arm_description/urdf/arm_description.urdf (robot description, URDF)
Before this commit: robot arm_description, 5 links, 4 joints
Links:
- added link world
Joints:
- added joint fixed: type fixed, parent world, child base_link

File: arm_description/urdf/test.urdf (robot description, URDF)
Before this commit: robot arm_description, 5 links, 4 joints
Links:
- added link world
