Commit message: Update easyarm仿真

File: easyarm_description/urdf/easyarm_description.urdf (robot description, URDF)
Before this commit: robot easyarm_description, 7 links, 6 joints
Joints:
- joint joint1: limit lower=-1.57 upper=1.57 effort=50 velocity=10 -> lower=-1.57 upper=1.57 effort=10 velocity=1
- joint joint2: limit lower=-1.57 upper=1.57 effort=50 velocity=10 -> lower=-1.57 upper=1.57 effort=10 velocity=1
- joint joint3: limit lower=-1.57 upper=1.57 effort=50 velocity=10 -> lower=-1.57 upper=1.57 effort=10 velocity=1
- joint joint4: limit lower=-1.57 upper=1.57 effort=50 velocity=10 -> lower=-1.57 upper=1.57 effort=10 velocity=1
